Commit message: 第一次跑起来后完善修改￥更改高精度地图

File: src/urdf/lexus_rx_450h_description/urdf/lexus_rx_450h_vehicle.urdf (robot description, URDF)
Before this commit: robot lexus_rx_450h, 3 links, 2 joints
Links:
- link base_link: geometry collision box size=1.6 1 1; visual mesh filename=package://lexus_rx_450h_description/meshes/LexusRX.obj scale=0.00045 0.0003 0.0005
Joints:
- joint lidar_front_joint: origin xyz=1.4 0 1.422 rpy=0.0215759 0.125004 0.111496 -> xyz=0.47 0 0.86 rpy=0.0215759 0.125004 0.111496
- joint lidar_rear_joint: origin xyz=0.1 0.01 1.422 rpy=0 0.146539 3.13 -> xyz=0.47 0 0.86 rpy=0.0215759 0.125004 0.111496
